File: distribution-amp.sch (KiCad schematic (older format))
At the start: 42 parts, among them J1 Conn_Coaxial, J2 Conn_Coaxial, J3 Conn_Coaxial, J4 Conn_Coaxial, J5 Conn_Coaxial, J6 PJ-037BH, U1 MC78M09_TO252, U2 MAX4022ESDT

Commit message: Add documentation
Other:
- note added: "Mounting Holes"
- note added: "Power supply: 12V - 15V DC, 100mA min."
- note added: "RF Input: 10dBm max into 50 Ohm.\nInput filter roll-off: -3dB @ 12Mhz"
- note added: "RF Output: 10dBm max. into 50 Ohm."
- note added: "open hardware"
- moved on the sheet: C1, C11, C2, C3, C4, D1, J4, J6, TP1, U1

Commit message: Documentation update
Other:
- note added: "RF Input: 10dBm max into 50 Ohm.\nInput filter cut-off: -3dB @ 13.8Mhz,\nroll-off: -38dB/octave"
- note removed: "RF Input: 10dBm max into 50 Ohm.\nInput filter roll-off: -3dB @ 12Mhz"
Changed lines of the file:
@@
 Power supply: 12V - 15V DC, 100mA min.
 Text Notes 1600 3500 0    50   ~ 0
-RF Input: 10dBm max into 50 Ohm.\nInput filter roll-off: -3dB @ 12Mhz
+RF Input: 10dBm max into 50 Ohm.\nInput filter cut-off: -3dB @ 13.8Mhz,\nroll-off: -38dB/octave
 Text Notes 9450 2650 0    50   ~ 0
 RF Output: 10dBm max. into 50 Ohm.
